File: board_design/mazeSolver.brd (EAGLE design)
At the start: 130 x 130 mm, 53 parts, among them IC1 L293DD, IC2 7805TV, IC3 CP2101, Q1 BC547, Q2 BC547, U1 MPU-9250, U2 AP1509-SOP8L, U3 ESP-WROOM-32, U4 GY-521MPU6050, U5 RST, U6 BOOT

Commit message: A lot of changes
Parts:
- removed IC3: CP2101, silabs-2:MLP28
- removed U1: MPU-9250, MPU-9250:QFN40P300X300X105-24N
- removed U4: GY-521MPU6050, gy-521:GY-521
- added C14: 22p, rcl:C1206
- added J1: (no value), SparkFun-Connectors:1X02
- added Q4: 32.768kHz, crystal-geyer_V1_0:3.2X2.5_KX-7
- added R18, R19, R20: 10k, rcl:R1206
- added U$11: BNO055, microbuilder:BNO055
- added U$9: T-PLUG_CONNECTOR, con-T-plug:T_PLUG_CONNECTOR
- added U7: INTERFACE-CP2102-GMR(QFN28), INTERFACE-CP2102-GMR_QFN28_:QFN28G_0.5-5X5MM
- C3: value 10n -> 0.1u
- C5: value 100n -> 0.1u
- C6: value 100n -> 22p
- moved C5 9.25 mm to (0.00, 5.08), turned to 270 degrees
- moved C3 2.84 mm to (7.62, -1.27), turned to 180 degrees
- moved C6 2.84 mm to (1.27, -5.08), turned to 90 degrees
- moved U$2 1.91 mm to (20.3, 5.08)
- moved U$3 1.75 mm to (-20.3, -4.92)
- moved C11 1.27 mm to (-44.5, 19.1)
Connections:
- removed net INT: U1.12, U3.10, U4.INT
- removed net N$22: C6.1, U1.10
- new net 3.3V: C3.2, U$11.28, U$11.3, U$11.4
- new net I2CADDR_3V: R18.1, U$11.17
- new net N$17: U$1.P$1, U$9.P$2
- new net N$19: J1.2, U3.12
- new net N$20: C6.2, Q4.3, U$11.27
- new net N$21: C14.2, Q4.1, U$11.26
- new net N$23: C5.2, U$11.9
- new net PS0_3V: R19.1, U$11.6
- new net PS1_3V: R20.1, U$11.5
- net +3V3: no longer C3.1, C5.1, U1.13, U1.8, U4.VCC
- net CTS: now also U7.23; no longer IC3.23
- net DTR: now also U7.28; no longer IC3.28
- net GND: now also C14.1, C3.1, C5.1, C6.1, J1.1, R18.2, R19.2, R20.2, U$11.10, U$11.15, U$11.16, U$11.18, U$11.2, U$11.25; no longer C3.2, C5.2, C6.2, IC3.3, IC3.EXP, IC3.M, U1.11, U1.18, U1.9, U4.GND
- net N$10: now also U7.8; no longer IC3.8
- net N$11: now also U7.6, U7.7; no longer IC3.6, IC3.7
- net N$8: now also U7.5; no longer IC3.5
- net N$9: now also U7.4; no longer IC3.4
- net RTS: now also U7.24; no longer IC3.24
- net RXD: now also U7.25; no longer IC3.25
- net SCL: now also U$11.19; no longer U1.23, U4.SCL
- net SDA: now also U$11.20; no longer U1.24, U4.SDA
- net TXD: now also U7.26; no longer IC3.26
- net VCC: now also U$9.P$1; no longer U$1.P$1
Routing:
- net N$19: track 0.00 -> 70.3 mm, vias 0 -> 2
- net INT: track 66.8 -> 0.00 mm, vias 1 -> 0
- net SDA: track 91.6 -> 75.9 mm
- net N$21: track 0.00 -> 13.6 mm
- net +3V3: track 511.7 -> 499.2 mm, vias 7 -> 4
- net SCL: track 92.5 -> 81.1 mm
- net N$20: track 0.00 -> 10.8 mm
- net 3.3V: track 0.00 -> 8.76 mm
- net N$17: track 0.00 -> 8.76 mm
- net RTS: track 55.2 -> 62.3 mm
- net N$10: track 20.2 -> 27.1 mm, vias 2 -> 0
- net GND: track 54.6 -> 48.4 mm, vias 9 -> 8
- net PS1_3V: track 0.00 -> 4.10 mm
- net N$22: track 3.52 -> 0.00 mm
- net N$8: track 14.0 -> 17.4 mm, vias 2 -> 0
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Other:
- board text added: "Design by: MM&MM"
- board text added: "aMazeSolver"

Commit message: PR review changes
Connections:
- net GND: now also U7.29
Routing:
- net GND: track 48.4 -> 60.8 mm

Commit message: PR review changes
Parts:
- moved C11 1.27 mm to (-44.5, 17.8)
Connections:
- removed net 3.3V: C3.2, U$11.28, U$11.3, U$11.4
- removed net N$11: C11.1, U7.6, U7.7
- net +3V3: now also C11.1, C3.2, IC1.20, U$11.28, U$11.3, U$11.4, U7.6, U7.7; no longer IC1.10
- net VCC: now also IC1.10; no longer IC1.20
Routing:
- net +3V3: track 499.2 -> 549.3 mm, vias 4 -> 7
- net 3.3V: track 8.76 -> 0.00 mm
- net N$11: track 3.37 -> 0.00 mm
- net VCC: track 185.1 -> 182.6 mm
- net N$10: track 27.1 -> 28.1 mm
- net GND: track 60.8 -> 61.3 mm, vias 8 -> 9
