File: board_design/mazeSolver.brd (EAGLE design)
At the start: 130 x 130 mm, 59 parts, among them IC1 L293DD, IC2 7805TV, Q1 BC547, Q2 BC547, Q4 32.768kHz, U2 AP1509-SOP8L, U3 ESP-WROOM-32, U5 RST, U6 BOOT, U7 INTERFACE-CP2102-GMR(QFN28)

Commit message: Board design changes
Parts:
- removed C11: 10u, rcl:C1206
- removed C12, C13, C4: 100n, rcl:C1206
- removed C14, C6: 22p, rcl:C1206
- removed C3, C5: 0.1u, rcl:C1206
- removed D2: (no value), diode:DO214AC
- removed Q1, Q2: BC547, semicon-smd-ipc:SOT23
- removed Q4: 32.768kHz, crystal-geyer_V1_0:3.2X2.5_KX-7
- removed R10, R16, R17, R7, R8, R9: 1k, rcl:R1206
- removed R11, R12, R15, R18, R19, R20: 10k, rcl:R1206
- removed SV1: (no value), con-lstb:MA04-1
- removed U$11: BNO055, microbuilder:BNO055
- removed U3: ESP-WROOM-32, esp32:ESP-WROOM-32
- removed U5: RST, Switches:SW4_236X236H5MM
- removed U6: BOOT, Switches:SW4_236X236H5MM
- removed U7: INTERFACE-CP2102-GMR(QFN28), INTERFACE-CP2102-GMR_QFN28_:QFN28G_0.5-5X5MM
- added F1: (no value), polyfuse:C1812K
- added F2: (no value), polyfuse:C1206K
- added R21: 10k, rcl:R1206
- added U1: ESP32-DEVKITC-32D, ESP32-DEVKITC-32D:MODULE_ESP32-DEVKITC-32D
- U$8: value MICRO-USB -> BNO055; device microusb:MICRO-USB -> bno055:BNO055
- moved U$8 67.1 mm to (1.27, -5.08), turned to 0 degrees
- moved IC1 2.84 mm to (1.27, 1.27)
- moved U$9 2.84 mm to (7.62, -41.9)
- moved C1 2.54 mm to (10.2, -48.3)
- moved C2 2.54 mm to (-14.0, -34.3)
- moved D1 2.54 mm to (-22.9, -43.2)
- moved IC2 2.54 mm to (0.00, -39.4)
- moved L1 2.54 mm to (-12.7, -48.3)
- moved U$1 2.54 mm to (16.5, -41.9)
- moved U2 2.54 mm to (0.00, -50.8)
Connections:
- removed net 3.3V: C3.2, U$11.28, U$11.3, U$11.4
- removed net CTS: U3.23, U7.23
- removed net DTR: Q2.2, R7.1, U7.28
- removed net EN: C4.2, Q1.3, R11.1, R16.2, U3.3
- removed net I2CADDR_3V: R18.1, U$11.17
- removed net IO0: Q2.3, R15.1, R17.2, U3.25
- removed net N$10: D2.A, U$8.1, U7.8
- removed net N$11: C11.1, U7.6, U7.7
- removed net N$12: Q1.1, R7.2
- removed net N$13: Q2.1, R8.2
- removed net N$14: C13.1, R16.1, U5.3, U5.4
- removed net N$15: C12.1, R17.1, U6.3, U6.4
- removed net N$16: R12.2, U3.24
- removed net N$20: C6.2, Q4.3, U$11.27
- removed net N$21: C14.2, Q4.1, U$11.26
- removed net N$23: C5.2, U$11.9
- removed net N$8: U$8.2, U7.5
- removed net N$9: U$8.3, U7.4
- removed net PS0_3V: R19.1, U$11.6
- removed net PS1_3V: R20.1, U$11.5
- removed net RTS: Q1.2, R8.1, U3.16, U7.24
- removed net RX: R9.2, U3.34
- removed net RXD: R10.1, SV1.2, U7.25
- removed net TX: R10.2, U3.35
- removed net TXD: R9.1, SV1.3, U7.26
- new net EXT_5V: U1.19
- new net N$22: F1.1, U$9.P$1
- new net N$24: C2.+, F2.1, L1.2, U2.3
- new net N$25: R21.1, U$4.3
- net +3V3: now also F2.2, R21.2, U$8.P$1, U1.1; no longer C2.+, L1.2, R11.2, R15.2, SV1.4, U2.3, U3.2
- net ENCA1: now also U1.7; no longer U3.7
- net ENCA2: now also U1.6; no longer U3.6
- net ENCB1: now also U1.5; no longer U3.5
- net ENCB2: now also U1.4; no longer U3.4
- net GND: now also U$8.P$2, U$8.P$5, U1.14, U1.20, U1.26; no longer C11.2, C12.2, C13.2, C14.1, C3.1, C4.1, C5.1, C6.1, R12.1, R18.2, R19.2, R20.2, SV1.1, U$11.10, U$11.15, U$11.16, U$11.18, U$11.2, U$11.25, U$4.3, U$8.5, U$8.GND1, U$8.GND2, U3.1, U3.15, U3.38, U3.GND, U5.1, U5.2, U6.1, U6.2
- net INA1: now also U1.31; no longer U3.27
- net INA2: now also U1.30; no longer U3.28
- net INB1: now also U1.28; no longer U3.30
- net INB2: now also U1.32; no longer U3.26
- net N$19: now also U1.12; no longer U3.12
- net SCL: now also U$8.P$4, U1.22; no longer U$11.19, U3.36
- net SDA: now also U$8.P$3, U1.25; no longer U$11.20, U3.33
- net VCC: now also F1.2; no longer D2.C, U$9.P$1
Routing:
- net +3V3: track 499.2 -> 318.1 mm, vias 4 -> 3
- net TXD: track 110.5 -> 0.00 mm, vias 2 -> 0
- net RXD: track 106.8 -> 0.00 mm, vias 2 -> 0
- net IO0: track 100.3 -> 0.00 mm, vias 4 -> 0
- net EN: track 66.7 -> 0.00 mm
- net RTS: track 62.3 -> 0.00 mm, vias 2 -> 0
- net CTS: track 56.5 -> 0.00 mm, vias 2 -> 0
- net GND: track 48.4 -> 0.00 mm, vias 8 -> 3
- net VCC: track 185.1 -> 146.3 mm, vias 1 -> 0
- net N$24: track 0.00 -> 28.5 mm
- net N$10: track 27.1 -> 0.00 mm
- net N$19: track 70.3 -> 43.9 mm, vias 2 -> 0
- net DTR: track 25.4 -> 0.00 mm
- net INA2: track 25.3 -> 7.39 mm, vias 1 -> 0
- net N$8: track 17.4 -> 0.00 mm
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