File: board_design/mazeSolver.sch (EAGLE design)
At the start: 53 parts, among them IC1 L293DD, IC2 7805TV, IC3 CP2101, Q1 BC547, Q2 BC547, U1 MPU-9250, U2 AP1509-SOP8L, U3 ESP-WROOM-32, U4 GY-521MPU6050, U5 RST, U6 BOOT

Commit message: A lot of changes
Parts:
- removed IC3: CP2101, silabs-2:CP2101
- removed U1: MPU-9250, MPU-9250:MPU-9250
- removed U4: GY-521MPU6050, gy-521:GY-521MPU6050
- added C14: 22p, rcl:C-EUC1206
- added J1: (no value), SparkFun-Connectors:CONN_02
- added Q4: 32.768kHz, crystal-geyer_V1_0:KX-7
- added R18, R19, R20: 10k, rcl:R-EU_R1206
- added U$11: BNO055, microbuilder:BNO055
- added U$9: T-PLUG_CONNECTOR, con-T-plug:T-PLUG_CONNECTOR
- added U7: INTERFACE-CP2102-GMR(QFN28), INTERFACE-CP2102-GMR_QFN28_:INTERFACE-CP2102-GMR(QFN28)
- C1: MF (none) -> RUBYCON; MPN (none) -> 100YXF100MEFC12.5X20; OC_FARNELL (none) -> 1144642
- C10, C11, C12, C13, C2, C4, C7, C8, C9, D1, D2, IC2, L1, Q1, Q2, R1, R10, R11, R12, R13, R14, R15, R16, R17, R2, R3, R4, R5, R6, R7, R8, R9, U$1, U$3, U$4, U$5, U$6, U$7, U$8, U2, U3, U5, U6: OC_FARNELL (none) -> unknown
- C3: value 10n -> 0.1u
- C5: value 100n -> 0.1u
- C6: value 100n -> 22p
Connections:
- removed net INT: U1.INT, U3.IO25, U4.INT
- removed net N$22: C6.1, U1.REGOUT
- new net 3.3V: C3.2, U$11.NBOOT_LOAD_PIN, U$11.VDD, U$11.VDDIO
- new net I2CADDR_3V: R18.1, U$11.COM3/I2C_ADDR
- new net N$17: U$1.P-1, U$9.P-2
- new net N$19: J1.2, U3.IO27
- new net N$20: C6.2, Q4.2, U$11.XIN32
- new net N$21: C14.2, Q4.1, U$11.XOUT32
- new net N$23: C5.2, U$11.CAP
- new net PS0_3V: R19.1, U$11.PS0
- new net PS1_3V: R20.1, U$11.PS1
- net +3V3: no longer C3.1, C5.1, U1.VDD, U1.VDDIO, U4.VCC
- net CTS: now also U7.CTS; no longer IC3.CTS
- net DTR: now also U7.DTR; no longer IC3.DTR
- net GND: now also C14.1, C3.1, C5.1, C6.1, J1.1, R18.2, R19.2, R20.2, U$11.COM2(GND), U$11.GND@1, U$11.GND@2, U$11.PIN10(GND), U$11.PIN15(GND), U$11.PIN16(GND); no longer C3.2, C5.2, C6.2, IC3.GND, IC3.GND@EXP, IC3.GND@M, U$8.GND, U1.AD0/SDO, U1.FSYNC, U1.GND, U4.GND
- net N$10: now also U7.VBUS; no longer IC3.VBUS
- net N$11: now also U7.REGIN, U7.VDD; no longer IC3.REGIN, IC3.VDD
- net N$8: now also U7.D-; no longer IC3.D-
- net N$9: now also U7.D+; no longer IC3.D+
- net RTS: now also U7.RTS; no longer IC3.RTS
- net RXD: now also U7.RXD; no longer IC3.RXD
- net SCL: now also U$11.COM1/SCL/RX; no longer U1.SCL/SCLK, U4.SCL
- net SDA: now also U$11.COM0/SDA/TX; no longer U1.SDA/SDI, U4.SDA
- net TXD: now also U7.TXD; no longer IC3.TXD
- net VCC: now also U$9.P-1; no longer U$1.P-1
Other:
- note removed: "IMU"

Commit message: PR review changes
Connections:
- net GND: now also U$8.GND, U7.GND@1
Changed lines of the file:
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@@
 <grid distance="0.1" unitdist="inch" unit="inch" style="lines" multiple="1" display="no" altdistance="0.01" altunitdist="inch" altunit="inch"/>
 <layers>
-<layer number="1" name="Top" color="4" fill="1" visible="yes" active="no"/>
-<layer number="2" name="Route2" color="16" fill="1" visible="yes" active="no"/>
-<layer number="3" name="Route3" color="17" fill="1" visible="yes" active="no"/>
-<layer number="4" name="Route4" color="18" fill="1" visible="yes" active="no"/>
-<layer number="5" name="Route5" color="19" fill="1" visible="yes" active="no"/>
-<layer number="6" name="Route6" color="25" fill="1" visible="yes" active="no"/>
-<layer number="7" name="Route7" color="26" fill="1" visible="yes" active="no"/>
-<layer number="8" name="Route8" color="27" fill="1" visible="yes" active="no"/>
-<layer number="9" name="Route9" color="28" fill="1" visible="yes" active="no"/>
-<layer number="10" name="Route10" color="29" fill="1" visible="yes" active="no"/>
-<layer number="11" name="Route11" color="30" fill="1" visible="yes" active="no"/>
-<layer number="12" name="Route12" color="20" fill="1" visible="yes" active="no"/>
-<layer number="13" name="Route13" color="21" fill="1" visible="yes" active="no"/>
-<layer number="14" name="Route14" color="22" fill="1" visible="yes" active="no"/>
-<layer number="15" name="Route15" color="23" fill="1" visible="yes" active="no"/>
-<layer number="16" name="Bottom" color="1" fill="1" visible="yes" active="no"/>
-<layer number="17" name="Pads" color="2" fill="1" visible="yes" active="no"/>
-<layer number="18" name="Vias" color="2" fill="1" visible="yes" active="no"/>
-<layer number="19" name="Unrouted" color="6" fill="1" visible="yes" active="no"/>
-<layer number="20" name="Dimension" color="24" fill="1" visible="yes" active="no"/>
-<layer number="21" name="tPlace" color="7" fill="1" visible="yes" active="no"/>
-<layer number="22" name="bPlace" color="7" fill="1" visible="yes" active="no"/>
-<layer number="23" name="tOrigins" color="15" fill="1" visible="yes" active="no"/>
-<layer number="24" name="bOrigins" color="15" fill="1" visible="yes" active="no"/>
-<layer number="25" name="tNames" color="7" fill="1" visible="yes" active="no"/>
-<layer number="26" name="bNames" color="7" fill="1" visible="yes" active="no"/>
-<layer number="27" name="tValues" color="7" fill="1" visible="yes" active="no"/>
-<layer number="28" name="bValues" color="7" fill="1" visible="yes" active="no"/>
+<layer number="1" name="Top" color="4" fill="1" visible="no" active="no"/>
+<layer number="2" name="Route2" color="16" fill="1" visible="no" active="no"/>
+<layer number="3" name="Route3" color="17" fill="1" visible="no" active="no"/>
+<layer number="4" name="Route4" color="18" fill="1" visible="no" active="no"/>
+<layer number="5" name="Route5" color="19" fill="1" visible="no" active="no"/>
+<layer number="6" name="Route6" color="25" fill="1" visible="no" active="no"/>
+<layer number="7" name="Route7" color="26" fill="1" visible="no" active="no"/>
+<layer number="8" name="Route8" color="27" fill="1" visible="no" active="no"/>
+<layer number="9" name="Route9" color="28" fill="1" visible="no" active="no"/>
+<layer number="10" name="Route10" color="29" fill="1" visible="no" active="no"/>
+<layer number="11" name="Route11" color="30" fill="1" visible="no" active="no"/>
+<layer number="12" name="Route12" color="20" fill="1" visible="no" active="no"/>
+<layer number="13" name="Route13" color="21" fill="1" visible="no" active="no"/>
+<layer number="14" name="Route14" color="22" fill="1" visible="no" active="no"/>
+<layer number="15" name="Route15" color="23" fill="1" visible="no" active="no"/>
+<layer number="16" name="Bottom" color="1" fill="1" visible="no" active="no"/>
+<layer number="17" name="Pads" color="2" fill="1" visible="no" active="no"/>
+<layer number="18" name="Vias" color="2" fill="1" visible="no" active="no"/>
+<layer number="19" name="Unrouted" color="6" fill="1" visible="no" active="no"/>
+<layer number="20" name="Dimension" color="24" fill="1" visible="no" active="no"/>
+<layer number="21" name="tPlace" color="7" fill="1" visible="no" active="no"/>
+<layer number="22" name="bPlace" color="7" fill="1" visible="no" active="no"/>
+<layer number="23" name="tOrigins" color="15" fill="1" visible="no" active="no"/>
+<layer number="24" name="bOrigins" color="15" fill="1" visible="no" active="no"/>
+<layer number="25" name="tNames" color="7" fill="1" visible="no" active="no"/>
+<layer number="26" name="bNames" color="7" fill="1" visible="no" active="no"/>
+<layer number="27" name="tValues" color="7" fill="1" visible="no" active="no"/>
+<layer number="28" name="bValues" color="7" fill="1" visible="no" active="no"/>
 <layer number="29" name="tStop" color="7" fill="3" visible="no" active="no"/>
 <layer number="30" name="bStop" color="7" fill="6" visible="no" active="no"/>
@@
 <layer number="35" name="tGlue" color="7" fill="4" visible="no" active="no"/>
 <layer number="36" name="bGlue" color="7" fill="5" visible="no" active="no"/>
-<layer number="37" name="tTest" color="7" fill="1" visible="yes" active="no"/>
-<layer number="38" name="bTest" color="7" fill="1" visible="yes" active="no"/>
+<layer number="37" name="tTest" color="7" fill="1" visible="no" active="no"/>
+<layer number="38" name="bTest" color="7" fill="1" visible="no" active="no"/>
 <layer number="39" name="tKeepout" color="4" fill="11" visible="no" active="no"/>
 <layer number="40" name="bKeepout" color="1" fill="11" visible="no" active="no"/>
@@
 <layer number="44" name="Drills" color="7" fill="1" visible="no" active="no"/>
 <layer number="45" name="Holes" color="7" fill="1" visible="no" active="no"/>
-<layer number="46" name="Milling" color="3" fill="1" visible="yes" active="no"/>
-<layer number="47" name="Measures" color="7" fill="1" visible="yes" active="no"/>
-<layer number="48" name="Document" color="7" fill="1" visible="yes" active="no"/>
-<layer number="49" name="Reference" color="7" fill="1" visible="yes" active="no"/>
-<layer number="50" name="dxf" color="7" fill="1" visible="yes" active="no"/>
-<layer number="51" name="tDocu" color="7" fill="1" visible="yes" active="no"/>
-<layer number="52" name="bDocu" color="7" fill="1" visible="yes" active="no"/>
-<layer number="53" name="tGND_GNDA" color="7" fill="9" visible="yes" active="no"/>
-<layer number="54" name="bGND_GNDA" color="1" fill="9" visible="yes" active="no"/>
-<layer number="56" name="wert" color="7" fill="1" visible="yes" active="no"/>
-<layer number="57" name="tCAD" color="7" fill="1" visible="yes" active="no"/>
-<layer number="59" name="tCarbon" color="7" fill="1" visible="yes" active="no"/>
-<layer number="60" name="bCarbon" color="7" fill="1" visible="yes" active="no"/>
+<layer number="46" name="Milling" color="3" fill="1" visible="no" active="no"/>
+<layer number="47" name="Measures" color="7" fill="1" visible="no" active="no"/>
+<layer number="48" name="Document" color="7" fill="1" visible="no" active="no"/>
+<layer number="49" name="Reference" color="7" fill="1" visible="no" active="no"/>
+<layer number="50" name="dxf" color="7" fill="1" visible="no" active="no"/>
+<layer number="51" name="tDocu" color="7" fill="1" visible="no" active="no"/>
+<layer number="52" name="bDocu" color="7" fill="1" visible="no" active="no"/>
+<layer number="53" name="tGND_GNDA" color="7" fill="9" visible="no" active="no"/>
+<layer number="54" name="bGND_GNDA" color="1" fill="9" visible="no" active="no"/>
+<layer number="56" name="wert" color="7" fill="1" visible="no" active="no"/>
+<layer number="57" name="tCAD" color="7" fill="1" visible="no" active="no"/>
+<layer number="59" name="tCarbon" color="7" fill="1" visible="no" active="no"/>
+<layer number="60" name="bCarbon" color="7" fill="1" visible="no" active="no"/>
 <layer number="88" name="SimResults" color="9" fill="1" visible="yes" active="yes"/>
 <layer number="89" name="SimProbes" color="9" fill="1" visible="yes" active="yes"/>
@@
 <attribute name="VALUE" x="223.52" y="124.46" size="1.778" layer="96"/>
 </instance>
-<instance part="GND28" gate="1" x="55.626" y="37.338" smashed="yes">
-<attribute name="VALUE" x="53.086" y="34.798" size="1.778" layer="96"/>
+<instance part="GND28" gate="1" x="68.326" y="42.418" smashed="yes">
+<attribute name="VALUE" x="65.786" y="39.878" size="1.778" layer="96"/>
 </instance>
 <instance part="GND31" gate="1" x="55.626" y="19.558" smashed="yes">
@@
 <wire x1="162.56" y1="114.3" x2="162.56" y2="111.76" width="0.1524" layer="91"/>
 </segment>
-</net>
+<segment>
+<pinref part="U$8" gate="G$1" pin="GND"/>
+<pinref part="GND31" gate="1" pin="GND"/>
+<wire x1="48.26" y1="30.48" x2="55.626" y2="30.48" width="0.1524" layer="91"/>
+<wire x1="55.626" y1="30.48" x2="55.626" y2="22.098" width="0.1524" layer="91"/>
+</segment>
+<segment>
+<pinref part="U7" gate="G$1" pin="GND@1"/>
+<pinref part="GND28" gate="1" pin="GND"/>
+<wire x1="63.5" y1="50.8" x2="68.326" y2="50.8" width="0.1524" layer="91"/>
+<wire x1="68.326" y1="50.8" x2="68.326" y2="44.958" width="0.1524" layer="91"/>
+</segment>
+</net>

Commit message: PR review changes
Connections:
- removed net 3.3V: C3.2, U$11.NBOOT_LOAD_PIN, U$11.VDD, U$11.VDDIO
- removed net N$11: C11.1, U7.REGIN, U7.VDD
- net +3V3: now also C11.1, C3.2, IC1.VSS, U$11.NBOOT_LOAD_PIN, U$11.VDD, U$11.VDDIO, U7.REGIN, U7.VDD; no longer IC1.VS
- net VCC: now also IC1.VS; no longer IC1.VSS
Changed lines of the file:
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@@
 <part name="GND9" library="supply1" library_urn="urn:adsk.eagle:library:371" deviceset="GND" device=""/>
 <part name="IC1" library="st-microelectronics" library_urn="urn:adsk.eagle:library:368" deviceset="L293DD" device="" package3d_urn="urn:adsk.eagle:package:26832/1" override_package3d_urn="urn:adsk.eagle:package:24674125/2" override_package_urn="urn:adsk.eagle:footprint:26750/1"/>
-<part name="P+3" library="supply1" library_urn="urn:adsk.eagle:library:371" deviceset="VCC" device=""/>
 <part name="GND10" library="supply1" library_urn="urn:adsk.eagle:library:371" deviceset="GND" device=""/>
 <part name="GND11" library="supply1" library_urn="urn:adsk.eagle:library:371" deviceset="GND" device=""/>
@@
 <part name="U$20" library="microbuilder" deviceset="GND" device=""/>
 <part name="U$21" library="microbuilder" deviceset="GND" device=""/>
-<part name="U$25" library="microbuilder" deviceset="3.3V" device=""/>
-<part name="U$26" library="microbuilder" deviceset="3.3V" device=""/>
 <part name="C3" library="rcl" library_urn="urn:adsk.eagle:library:334" deviceset="C-EU" device="C1206" package3d_urn="urn:adsk.eagle:package:23618/2" value="0.1u"/>
 <part name="C5" library="rcl" library_urn="urn:adsk.eagle:library:334" deviceset="C-EU" device="C1206" package3d_urn="urn:adsk.eagle:package:23618/2" value="0.1u"/>
@@
 <part name="U$2" library="pololu_encoder" deviceset="POLOLU_ENCODER" device="" override_package3d_urn="urn:adsk.eagle:package:24685780/2" override_package_urn="urn:adsk.eagle:footprint:24685781/1"/>
 <part name="Q4" library="crystal-geyer_V1_0" library_urn="urn:adsk.eagle:library:203" deviceset="KX" device="-7" package3d_urn="urn:adsk.eagle:package:11924/1" value="32.768kHz"/>
+<part name="P+3" library="supply1" library_urn="urn:adsk.eagle:library:371" deviceset="VCC" device=""/>
 </parts>
 <sheets>
@@
 <attribute name="VALUE" x="182.88" y="109.22" size="1.778" layer="96"/>
 </instance>
-<instance part="P+3" gate="VCC" x="210.82" y="149.86" smashed="yes">
-<attribute name="VALUE" x="213.36" y="152.4" size="1.778" layer="96" rot="R180"/>
-</instance>
 <instance part="GND10" gate="1" x="177.8" y="106.68" smashed="yes">
 <attribute name="VALUE" x="175.26" y="104.14" size="1.778" layer="96"/>
@@
 </instance>
 <instance part="U$2" gate="G$1" x="193.04" y="81.28" smashed="yes"/>
+<instance part="P+3" gate="VCC" x="177.8" y="152.4" smashed="yes">
+<attribute name="VALUE" x="175.26" y="149.86" size="1.778" layer="96" rot="R90"/>
+</instance>
 </instances>
 <busses>
@@
 </segment>
 <segment>
-<pinref part="IC1" gate="G$1" pin="VSS"/>
-<pinref part="P+3" gate="VCC" pin="VCC"/>
-<wire x1="205.74" y1="147.32" x2="210.82" y2="147.32" width="0.1524" layer="91"/>
-</segment>
-<segment>
 <pinref part="P+4" gate="VCC" pin="VCC"/>
 <wire x1="198.12" y1="88.9" x2="213.36" y2="88.9" width="0.1524" layer="91"/>
@@
 <pinref part="P+2" gate="VCC" pin="VCC"/>
 <wire x1="33.02" y1="86.36" x2="40.64" y2="86.36" width="0.1524" layer="91"/>
+</segment>
+<segment>
+<pinref part="P+3" gate="VCC" pin="VCC"/>
+<pinref part="IC1" gate="G$1" pin="VS"/>
+<wire x1="177.8" y1="149.86" x2="177.8" y2="147.32" width="0.1524" layer="91"/>
+<wire x1="177.8" y1="147.32" x2="180.34" y2="147.32" width="0.1524" layer="91"/>
 </segment>
 </net>
@@
 </segment>
 <segment>
-<pinref part="IC1" gate="G$1" pin="VS"/>
-<wire x1="180.34" y1="147.32" x2="175.26" y2="147.32" width="0.1524" layer="91"/>
-<label x="172.72" y="147.32" size="1.778" layer="95"/>
-</segment>
-<segment>
 <pinref part="IC1" gate="G$1" pin="EN1"/>
 <wire x1="180.34" y1="139.7" x2="175.26" y2="139.7" width="0.1524" layer="91"/>
@@
 <wire x1="81.28" y1="76.2" x2="88.9" y2="76.2" width="0.1524" layer="91"/>
 <label x="86.36" y="76.2" size="1.778" layer="95"/>
+</segment>
+<segment>
+<pinref part="IC1" gate="G$1" pin="VSS"/>
+<wire x1="205.74" y1="147.32" x2="210.82" y2="147.32" width="0.1524" layer="91"/>
+<label x="208.28" y="147.32" size="1.778" layer="95"/>
 </segment>
 </net>
@@
 <label x="144.78" y="73.66" size="1.778" layer="95"/>
 </segment>
+<segment>
+<pinref part="U7" gate="G$1" pin="REGIN"/>
+<pinref part="C11" gate="G$1" pin="1"/>
+<wire x1="35.56" y1="40.64" x2="35.56" y2="38.1" width="0.1524" layer="91"/>
+<wire x1="35.56" y1="38.1" x2="35.56" y2="30.48" width="0.1524" layer="91"/>
+<wire x1="35.56" y1="30.48" x2="25.4" y2="30.48" width="0.1524" layer="91"/>
+<pinref part="U7" gate="G$1" pin="VDD"/>
+<wire x1="38.1" y1="40.64" x2="38.1" y2="38.1" width="0.1524" layer="91"/>
+<wire x1="38.1" y1="38.1" x2="35.56" y2="38.1" width="0.1524" layer="91"/>
+<junction x="35.56" y="38.1"/>
+<label x="27.94" y="30.48" size="1.778" layer="95"/>
+</segment>
 </net>
 <net name="INA1" class="0">
@@
 <pinref part="D2" gate="G$1" pin="A"/>
 <junction x="22.86" y="35.56"/>
-</segment>
-</net>
-<net name="N$11" class="0">
-<segment>
-<pinref part="U7" gate="G$1" pin="REGIN"/>
-<pinref part="C11" gate="G$1" pin="1"/>
-<wire x1="35.56" y1="40.64" x2="35.56" y2="38.1" width="0.1524" layer="91"/>
-<wire x1="35.56" y1="38.1" x2="35.56" y2="30.48" width="0.1524" layer="91"/>
-<wire x1="35.56" y1="30.48" x2="25.4" y2="30.48" width="0.1524" layer="91"/>
-<pinref part="U7" gate="G$1" pin="VDD"/>
-<wire x1="38.1" y1="40.64" x2="38.1" y2="38.1" width="0.1524" layer="91"/>
-<wire x1="38.1" y1="38.1" x2="35.56" y2="38.1" width="0.1524" layer="91"/>
-<junction x="35.56" y="38.1"/>
 </segment>
 </net>
@@
 <attribute name="VALUE" x="142.24" y="115.316" size="1.27" layer="96" rot="R90"/>
 </instance>
-<instance part="U$25" gate="G$1" x="53.34" y="147.32" smashed="yes">
-<attribute name="VALUE" x="51.816" y="148.336" size="1.27" layer="96"/>
-</instance>
-<instance part="U$26" gate="G$1" x="101.6" y="111.76" smashed="yes" rot="R270">
-<attribute name="VALUE" x="102.616" y="113.284" size="1.27" layer="96" rot="R270"/>
-</instance>
 <instance part="C3" gate="G$1" x="45.72" y="142.24" smashed="yes" rot="R90">
 <attribute name="NAME" x="45.339" y="143.764" size="1.778" layer="95" rot="R90"/>
@@
 </segment>
 </net>
-<net name="3.3V" class="0">
+<net name="SDA" class="0">
+<segment>
+<pinref part="U$11" gate="G$1" pin="COM0/SDA/TX"/>
+<wire x1="96.52" y1="142.24" x2="101.6" y2="142.24" width="0.1524" layer="91"/>
+<label x="99.06" y="142.24" size="1.778" layer="95"/>
+</segment>
+</net>
+<net name="SCL" class="0">
+<segment>
+<pinref part="U$11" gate="G$1" pin="COM1/SCL/RX"/>
+<wire x1="96.52" y1="139.7" x2="101.6" y2="139.7" width="0.1524" layer="91"/>
+<label x="99.06" y="139.7" size="1.778" layer="95"/>
+</segment>
+</net>
+<net name="+3V3" class="0">
 <segment>
 <pinref part="U$11" gate="G$1" pin="VDDIO"/>
-<pinref part="U$25" gate="G$1" pin="3.3V"/>
 <wire x1="55.88" y1="139.7" x2="53.34" y2="139.7" width="0.1524" layer="91"/>
 <wire x1="53.34" y1="139.7" x2="53.34" y2="142.24" width="0.1524" layer="91"/>
@@
 <wire x1="50.8" y1="142.24" x2="53.34" y2="142.24" width="0.1524" layer="91"/>
 <pinref part="C3" gate="G$1" pin="2"/>
+<label x="50.8" y="144.78" size="1.778" layer="95"/>
 </segment>
 <segment>
 <pinref part="U$11" gate="G$1" pin="NBOOT_LOAD_PIN"/>
-<pinref part="U$26" gate="G$1" pin="3.3V"/>
-<wire x1="96.52" y1="111.76" x2="99.06" y2="111.76" width="0.1524" layer="91"/>
-</segment>
-</net>
-<net name="SDA" class="0">
-<segment>
-<pinref part="U$11" gate="G$1" pin="COM0/SDA/TX"/>
-<wire x1="96.52" y1="142.24" x2="101.6" y2="142.24" width="0.1524" layer="91"/>
-<label x="99.06" y="142.24" size="1.778" layer="95"/>
-</segment>
-</net>
-<net name="SCL" class="0">
-<segment>
-<pinref part="U$11" gate="G$1" pin="COM1/SCL/RX"/>
-<wire x1="96.52" y1="139.7" x2="101.6" y2="139.7" width="0.1524" layer="91"/>
-<label x="99.06" y="139.7" size="1.778" layer="95"/>
-</segment>
-</net>
+<wire x1="96.52" y1="111.76" x2="101.6" y2="111.76" width="0.1524" layer="91"/>
+<label x="96.52" y="111.76" size="1.778" layer="95"/>
+</segment>
+</net>
