File: board_design/mazeSolver.sch (EAGLE design)
At the start: 59 parts, among them IC1 L293DD, IC2 7805TV, Q1 BC547, Q2 BC547, Q4 32.768kHz, U2 AP1509-SOP8L, U3 ESP-WROOM-32, U5 RST, U6 BOOT, U7 INTERFACE-CP2102-GMR(QFN28)

Commit message: Board design changes
Parts:
- removed C11: 10u, rcl:C-EUC1206
- removed C12, C13, C4: 100n, rcl:C-EUC1206
- removed C14, C6: 22p, rcl:C-EUC1206
- removed C3, C5: 0.1u, rcl:C-EUC1206
- removed D2: (no value), diode:DIODE-DO214AC
- removed Q1, Q2: BC547, semicon-smd-ipc:NPN-TRANSISTOR_SOT23
- removed Q4: 32.768kHz, crystal-geyer_V1_0:KX-7
- removed R10, R16, R17, R7, R8, R9: 1k, rcl:R-EU_R1206
- removed R11, R12, R15, R18, R19, R20: 10k, rcl:R-EU_R1206
- removed SV1: (no value), con-lstb:MA04-1
- removed U$11: BNO055, microbuilder:BNO055
- removed U3: ESP-WROOM-32, esp32:ESP-WROOM-32
- removed U5: RST, Switches:4-1437565-1
- removed U6: BOOT, Switches:4-1437565-1
- removed U7: INTERFACE-CP2102-GMR(QFN28), INTERFACE-CP2102-GMR_QFN28_:INTERFACE-CP2102-GMR(QFN28)
- added F1: (no value), polyfuse:195591812
- added F2: (no value), polyfuse:195591206
- added R21: 10k, rcl:R-EU_R1206
- added U1: ESP32-DEVKITC-32D, ESP32-DEVKITC-32D:ESP32-DEVKITC-32D
- U$8: value MICRO-USB -> BNO055; device microusb:MICRO-USB -> bno055:BNO055; OC_FARNELL unknown -> (none)
Connections:
- removed net 3.3V: C3.2, U$11.NBOOT_LOAD_PIN, U$11.VDD, U$11.VDDIO
- removed net CTS: U3.IO15, U7.CTS
- removed net DTR: Q2.E, R7.1, U7.DTR
- removed net EN: C4.2, Q1.C, R11.1, R16.2, U3.EN
- removed net I2CADDR_3V: R18.1, U$11.COM3/I2C_ADDR
- removed net IO0: Q2.C, R15.1, R17.2, U3.IO0
- removed net N$10: D2.A, U$8.VCC, U7.VBUS
- removed net N$11: C11.1, U7.REGIN, U7.VDD
- removed net N$12: Q1.B, R7.2
- removed net N$13: Q2.B, R8.2
- removed net N$14: C13.1, R16.1, U5.3, U5.4
- removed net N$15: C12.1, R17.1, U6.3, U6.4
- removed net N$16: R12.2, U3.IO2
- removed net N$20: C6.2, Q4.2, U$11.XIN32
- removed net N$21: C14.2, Q4.1, U$11.XOUT32
- removed net N$23: C5.2, U$11.CAP
- removed net N$8: U$8.D-, U7.D-
- removed net N$9: U$8.D+, U7.D+
- removed net PS0_3V: R19.1, U$11.PS0
- removed net PS1_3V: R20.1, U$11.PS1
- removed net RTS: Q1.E, R8.1, U3.IO13, U7.RTS
- removed net RX: R9.2, U3.RXD0
- removed net RXD: R10.1, SV1.2, U7.RXD
- removed net TX: R10.2, U3.TXD0
- removed net TXD: R9.1, SV1.3, U7.TXD
- new net N$22: F1.1, U$9.P-1
- new net N$24: C2.+, F2.1, L1.2, U2.FB
- new net N$25: R21.1, U$4.RST
- net +3V3: now also F2.2, R21.2, U$8.VCC, U1.3V3; no longer C2.+, L1.2, R11.2, R15.2, SV1.4, U2.FB, U3.3V3
- net ENCA1: now also U1.IO32; no longer U3.IO35
- net ENCA2: now also U1.IO35; no longer U3.IO34
- net ENCB1: now also U1.IO34; no longer U3.SENSOR_VN
- net ENCB2: now also U1.SENSOR_VN; no longer U3.SENSOR_VP
- net GND: now also U$8.GND, U$8.I2C, U1.GND1, U1.GND2, U1.GND3; no longer C11.2, C12.2, C13.2, C14.1, C3.1, C4.1, C5.1, C6.1, R12.1, R18.2, R19.2, R20.2, SV1.1, U$11.COM2(GND), U$11.GND@1, U$11.GND@2, U$11.PIN10(GND), U$11.PIN15(GND), U$11.PIN16(GND), U$4.RST, U3.GND@1, U3.GND@2, U3.GND@3, U3.GND@4, U5.1, U5.2, U6.1, U6.2
- net INA1: now also U1.IO16; no longer U3.IO16
- net INA2: now also U1.IO17; no longer U3.IO17
- net INB1: now also U1.IO18; no longer U3.IO18
- net INB2: now also U1.IO4; no longer U3.IO4
- net N$19: now also U1.IO14; no longer U3.IO27
- net SCL: now also U$8.LRX, U1.IO22; no longer U$11.COM1/SCL/RX, U3.IO22
- net SDA: now also U$8.ATX, U1.IO21; no longer U$11.COM0/SDA/TX, U3.IO21
- net VCC: now also F1.2; no longer D2.C, U$9.P-1
Other:
- note added: "IMU"
- note removed: "USB to TTL"
- note removed: "switch controls"
- moved on the sheet: C1, C2, D1, IC2, J1, L1, U2
